Commit message: feat: agregado de brida y base del robot al package. Mejoras estéticas.

File: mycobot_description/urdf/mycobot_320_pi_2022/mycobot_320_pi_2022DH.urdf (robot description, URDF)
Before this commit: robot firefighter, 14 links, 13 joints
Links:
- added link base_flange; collision mesh filename=package://mycobot_description/urdf/mycobot_320_pi_2022/base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 scale=0.001 0.001 0.001; visual mesh filename=package://mycobot_description/urdf/mycobot_320_pi_2022/base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 scale=0.001 0.001 0.001
- added link base_mesa; collision mesh filename=package://mycobot_description/urdf/mycobot_320_pi_2022/base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 scale=0.001 0.001 0.001; visual mesh filename=package://mycobot_description/urdf/mycobot_320_pi_2022/base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 scale=0.001 0.001 0.001
Joints:
- added joint base_to_flange: type fixed, parent base, child base_flange, origin xyz=0 0 0.0 rpy=0 0 0
- added joint flange_to_mesa: type fixed, parent base_flange, child base_mesa, origin xyz=0 0 0.0 rpy=0 0 0
